File: hardware/SensorPod/PCB/SensorPod-Board.kicad_sch (KiCad schematic)
At the start: 17 parts, among them J1 EXT, J2 EXT I2C, J3 Reset, J4 DC 5-15v, J5 Power select, Q1 TP0610L, U1 Pico W, U2 SCD30, U3 LM1117-3.3

Commit message: Fixed up paths for extra device symbols/models. Swapped HIB design over to Pico W footprint
Parts:
- U1: footprint RPi_Pico:RPi_PicoW_SMD_TH -> RPi_PicoW:RPi_Pico_SMD_TH; symbol RPi_Pico:PicoW -> PicoW:PicoW
Changed lines of the file:
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@@
     (pin "1")
   )
-  (symbol (lib_id "RPi_Pico:PicoW") (at 165.1 104.14 0) (unit 1)
+  (symbol (lib_id "PicoW:PicoW") (at 165.1 104.14 0) (unit 1)
     (in_bom yes) (on_board yes) (fields_autoplaced)
     (property "Reference" "U1" (id 0) (at 165.1 72.39 0))
     (property "Value" "Pico W" (id 1) (at 165.1 74.93 0))
-    (property "Footprint" "RPi_Pico:RPi_PicoW_SMD_TH" (id 2) (at 165.1 104.14 90)
+    (property "Footprint" "RPi_PicoW:RPi_Pico_SMD_TH" (id 2) (at 165.1 104.14 90)
       (effects (font (size 1.27 1.27)) hide)
     )
@@
     )
     (path "/edc16dc7-3087-489e-9478-e0104b4d8c62"
-      (reference "U1") (unit 1) (value "Pico W") (footprint "RPi_Pico:RPi_PicoW_SMD_TH")
+      (reference "U1") (unit 1) (value "Pico W") (footprint "RPi_PicoW:RPi_Pico_SMD_TH")
     )
     (path "/a18a804a-71b6-4fa4-a9fe-740ba1a67f07"
